File: spinnybot-motherboad/power.kicad_sch (KiCad schematic)
At the start: 26 parts, among them J1 +12V, J2 GND, J3 POWER SW1, J4 POWER SW2, Q1 SISA96DN, Q2 Q_NMOS_DGS, Q4 SISA96DN, U2 LM1117-3.3

Commit message: fixed some reference designators so the layout isn't broken
Parts:
- renumbered C2 to C1, C3 to C2, C4 to C3, C5 to C4, C1 to C5, J4 to J11, J2 to J5, J3 to J9, Q4 to Q2, Q2 to Q4, R3 to R1, R4 to R2, R5 to R3, R6 to R4, R7 to R5, R1 to R6, R2 to R7, R8 to R9, U2 to U1
Other:
- note added: "ADJUST VALUES OF R6, R7, AND C5 AS NEEDED"
- note removed: "ADJUST VALUES OF R1, R2, AND C1 AS NEEDED"
Changed lines of the file:
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@@
     (effects (font (size 1.27 1.27)) (justify right bottom))
   )
-  (text "ADJUST VALUES OF R1, R2, AND C1\nAS NEEDED" (at 185.42 60.96 0)
+  (text "ADJUST VALUES OF R6, R7, AND C5\nAS NEEDED" (at 185.42 60.96 0)
     (effects (font (size 1.27 1.27)) (justify left bottom))
   )
@@
   (symbol (lib_id "Connector_Generic:Conn_01x01") (at 68.58 30.48 90) (unit 1)
     (in_bom yes) (on_board yes)
-    (property "Reference" "J2" (id 0) (at 68.5038 24.4602 90))
+    (property "Reference" "J5" (id 0) (at 68.5038 24.4602 90))
     (property "Value" "GND" (id 1) (at 68.5038 26.7716 90))
     (property "Footprint" "custom:Stitched_SolderWirePad_1x01_SMD_5x10mm" (id 2) (at 68.58 30.48 0)
@@
   (symbol (lib_id "Device:C") (at 53.34 35.56 270) (unit 1)
     (in_bom yes) (on_board yes)
-    (property "Reference" "C3" (id 0) (at 53.34 41.91 90))
+    (property "Reference" "C2" (id 0) (at 53.34 41.91 90))
     (property "Value" "10u" (id 1) (at 53.34 39.37 90))
     (property "Footprint" "Capacitor_SMD:C_0805_2012Metric_Pad1.18x1.45mm_HandSolder" (id 2) (at 49.53 36.5252 0)
@@
   (symbol (lib_id "Device:R") (at 47.625 76.2 0) (unit 1)
     (in_bom yes) (on_board yes)
-    (property "Reference" "R3" (id 0) (at 50.165 75.5649 0)
+    (property "Reference" "R1" (id 0) (at 50.165 75.5649 0)
       (effects (font (size 1.27 1.27)) (justify left))
     )
@@
   (symbol (lib_id "spinnybot:SISA96DN") (at 245.11 93.98 0) (unit 1)
     (in_bom yes) (on_board yes)
-    (property "Reference" "Q4" (id 0) (at 245.11 83.82 0))
+    (property "Reference" "Q2" (id 0) (at 245.11 83.82 0))
     (property "Value" "SISA96DN" (id 1) (at 245.11 86.36 0))
     (property "Footprint" "Package_SO:Vishay_PowerPAK_1212-8_Single" (id 2) (at 245.11 102.87 0)
@@
   (symbol (lib_id "Device:R") (at 212.09 39.37 0) (unit 1)
     (in_bom yes) (on_board yes) (fields_autoplaced)
-    (property "Reference" "R1" (id 0) (at 214.63 38.0999 0)
+    (property "Reference" "R6" (id 0) (at 214.63 38.0999 0)
       (effects (font (size 1.27 1.27)) (justify left))
     )
@@
   (symbol (lib_id "Device:R") (at 151.13 27.94 270) (unit 1)
     (in_bom yes) (on_board yes)
-    (property "Reference" "R5" (id 0) (at 151.13 33.02 90))
+    (property "Reference" "R3" (id 0) (at 151.13 33.02 90))
     (property "Value" "1K" (id 1) (at 151.13 30.48 90))
     (property "Footprint" "Resistor_SMD:R_0805_2012Metric_Pad1.20x1.40mm_HandSolder" (id 2) (at 151.13 26.162 90)
@@
   (symbol (lib_id "Device:R") (at 243.84 38.1 180) (unit 1)
     (in_bom yes) (on_board yes) (fields_autoplaced)
-    (property "Reference" "R8" (id 0) (at 246.38 36.8299 0)
+    (property "Reference" "R9" (id 0) (at 246.38 36.8299 0)
       (effects (font (size 1.27 1.27)) (justify right))
     )
@@
   (symbol (lib_id "Device:R") (at 219.71 46.99 90) (unit 1)
     (in_bom yes) (on_board yes) (fields_autoplaced)
-    (property "Reference" "R2" (id 0) (at 219.71 40.64 90))
+    (property "Reference" "R7" (id 0) (at 219.71 40.64 90))
     (property "Value" "2k" (id 1) (at 219.71 43.18 90))
     (property "Footprint" "Resistor_SMD:R_0805_2012Metric_Pad1.20x1.40mm_HandSolder" (id 2) (at 219.71 48.768 90)
@@
   (symbol (lib_id "Device:R") (at 151.13 38.1 270) (unit 1)
     (in_bom yes) (on_board yes)
-    (property "Reference" "R6" (id 0) (at 151.13 43.18 90))
+    (property "Reference" "R4" (id 0) (at 151.13 43.18 90))
     (property "Value" "301" (id 1) (at 151.13 40.64 90))
     (property "Footprint" "Resistor_SMD:R_0805_2012Metric_Pad1.20x1.40mm_HandSolder" (id 2) (at 151.13 36.322 90)
@@
   (symbol (lib_id "Device:R") (at 47.625 83.82 0) (unit 1)
     (in_bom yes) (on_board yes)
-    (property "Reference" "R4" (id 0) (at 50.165 83.1849 0)
+    (property "Reference" "R2" (id 0) (at 50.165 83.1849 0)
       (effects (font (size 1.27 1.27)) (justify left))
     )
@@
   (symbol (lib_id "Device:C") (at 37.465 83.82 0) (unit 1)
     (in_bom yes) (on_board yes)
-    (property "Reference" "C2" (id 0) (at 41.275 83.1849 0)
+    (property "Reference" "C1" (id 0) (at 41.275 83.1849 0)
       (effects (font (size 1.27 1.27)) (justify left))
     )
@@
   (symbol (lib_id "Regulator_Linear:LM1117-3.3") (at 81.28 50.8 0) (unit 1)
     (in_bom yes) (on_board yes)
-    (property "Reference" "U2" (id 0) (at 81.28 44.6532 0))
+    (property "Reference" "U1" (id 0) (at 81.28 44.6532 0))
     (property "Value" "LM1117-3.3" (id 1) (at 81.28 46.9646 0))
     (property "Footprint" "Package_TO_SOT_SMD:SOT-223-3_TabPin2" (id 2) (at 81.28 50.8 0)
@@
   (symbol (lib_id "Device:Q_NMOS_DGS") (at 241.3 46.99 0) (unit 1)
     (in_bom yes) (on_board yes) (fields_autoplaced)
-    (property "Reference" "Q2" (id 0) (at 247.65 45.7199 0)
+    (property "Reference" "Q4" (id 0) (at 247.65 45.7199 0)
       (effects (font (size 1.27 1.27)) (justify left))
     )
@@
   (symbol (lib_id "Connector_Generic:Conn_01x02") (at 194.31 40.64 0) (unit 1)
     (in_bom yes) (on_board yes) (fields_autoplaced)
-    (property "Reference" "J4" (id 0) (at 196.85 40.6399 0)
+    (property "Reference" "J11" (id 0) (at 196.85 40.6399 0)
       (effects (font (size 1.27 1.27)) (justify left))
     )
@@
   (symbol (lib_id "Connector_Generic:Conn_01x02") (at 194.31 31.75 0) (unit 1)
     (in_bom yes) (on_board yes) (fields_autoplaced)
-    (property "Reference" "J3" (id 0) (at 196.85 31.7499 0)
+    (property "Reference" "J9" (id 0) (at 196.85 31.7499 0)
       (effects (font (size 1.27 1.27)) (justify left))
     )
@@
   (symbol (lib_id "Device:C") (at 226.06 53.34 180) (unit 1)
     (in_bom yes) (on_board yes) (fields_autoplaced)
-    (property "Reference" "C1" (id 0) (at 229.87 52.0699 0)
+    (property "Reference" "C5" (id 0) (at 229.87 52.0699 0)
       (effects (font (size 1.27 1.27)) (justify right))
     )
@@
   (symbol (lib_id "Device:C") (at 91.44 54.61 0) (unit 1)
     (in_bom yes) (on_board yes)
-    (property "Reference" "C5" (id 0) (at 95.25 53.9749 0)
+    (property "Reference" "C4" (id 0) (at 95.25 53.9749 0)
       (effects (font (size 1.27 1.27)) (justify left))
     )
@@
   (symbol (lib_id "Device:R") (at 151.13 48.26 270) (unit 1)
     (in_bom yes) (on_board yes)
-    (property "Reference" "R7" (id 0) (at 151.13 53.34 90))
+    (property "Reference" "R5" (id 0) (at 151.13 53.34 90))
     (property "Value" "130" (id 1) (at 151.13 50.8 90))
     (property "Footprint" "Resistor_SMD:R_0805_2012Metric_Pad1.20x1.40mm_HandSolder" (id 2) (at 151.13 46.482 90)
@@
   (symbol (lib_id "Device:C") (at 70.485 60.325 0) (unit 1)
     (in_bom yes) (on_board yes)
-    (property "Reference" "C4" (id 0) (at 73.025 62.2299 0)
-      (effects (font (size 1.27 1.27)) (justify left))
-    )
+    (property "Reference" "C3" (id 0) (at 73.025 62.2299 0)
+      (effects (font (size 1.27 1.27)) (justify left))
+    )

Commit message: Changed values for power RC circuit
Parts:
- R7: value 2k -> 150k
Other:
- note removed: "ADJUST VALUES OF R6, R7, AND C5 AS NEEDED"
Changed lines of the file:
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@@
     (effects (font (size 1.27 1.27)) (justify right bottom))
-  )
-  (text "ADJUST VALUES OF R6, R7, AND C5\nAS NEEDED" (at 185.42 60.96 0)
-    (effects (font (size 1.27 1.27)) (justify left bottom))
   )
   (text "MAKE SURE THIS MOSFET'S\nPINS MATCH THE FOOTPRINT" (at 238.76 63.5 0)
@@
     (in_bom yes) (on_board yes) (fields_autoplaced)
     (property "Reference" "R7" (id 0) (at 219.71 40.64 90))
-    (property "Value" "2k" (id 1) (at 219.71 43.18 90))
+    (property "Value" "150k" (id 1) (at 219.71 43.18 90))
     (property "Footprint" "Resistor_SMD:R_0805_2012Metric_Pad1.20x1.40mm_HandSolder" (id 2) (at 219.71 48.768 90)
       (effects (font (size 1.27 1.27)) hide)

Commit message: Removed buck converter PS1, voltage sense divider, and motor connections. Added encoder connectors
Parts:
- removed C1: 10u, Capacitor_SMD:C_1206_3216Metric_Pad1.33x1.80mm_HandSolder, symbol Device:C
- removed C2: 10u, Capacitor_SMD:C_0805_2012Metric_Pad1.18x1.45mm_HandSolder, symbol Device:C
- removed J1: +12V, Connector_Wire:SolderWirePad_1x01_SMD_5x10mm, symbol Connector_Generic:Conn_01x01
- removed J5: GND, custom:Stitched_SolderWirePad_1x01_SMD_5x10mm, symbol Connector_Generic:Conn_01x01
- removed PS1: R-78E5.0-1.0, R-78E5:CONV_R-78E5.0-1.0, symbol R-78E5.0-1.0:R-78E5.0-1.0
- removed R1: 3.92K, Resistor_SMD:R_0805_2012Metric_Pad1.20x1.40mm_HandSolder, symbol Device:R
- removed R2: 909, Resistor_SMD:R_0805_2012Metric_Pad1.20x1.40mm_HandSolder, symbol Device:R

Commit message: Made and imported ESC footprint, added 10 pin JST connector symbol and footprint, updated Q2 FET to control ESC power
Connections:
- net MOTOR_NEG renamed ESC_GND
Changed lines of the file:
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@@
     (effects (font (size 1.27 1.27)) (justify left))
   )
-  (hierarchical_label "MOTOR_NEG" (shape input) (at 228.6 81.28 180)
+  (hierarchical_label "ESC_GND" (shape input) (at 228.6 81.28 180)
     (effects (font (size 1.27 1.27)) (justify right))
   )
