File: spinnybot-motherboad/power.kicad_sch (KiCad schematic)
At the start: 26 parts, among them J10 ESC_POS, J11 POWER SW2, J15 BAT_GND, J16 ESC_GND, J8 BAT_POS, J9 POWER SW1, Q1 SISA96DN, Q2 SISA96DN, Q4 BC846, U1 LM1117-3.3

Commit message: Updated voltage divider on power circuit
Parts:
- R10: value 10K -> 100K
- R7: value 150k -> 15k
Changed lines of the file:
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@@
     (in_bom yes) (on_board yes) (fields_autoplaced)
     (property "Reference" "R10" (id 0) (at 240.03 40.64 90))
-    (property "Value" "10K" (id 1) (at 240.03 43.18 90))
+    (property "Value" "100K" (id 1) (at 240.03 43.18 90))
     (property "Footprint" "Resistor_SMD:R_0805_2012Metric_Pad1.20x1.40mm_HandSolder" (id 2) (at 240.03 48.768 90)
       (effects (font (size 1.27 1.27)) hide)
@@
     (in_bom yes) (on_board yes) (fields_autoplaced)
     (property "Reference" "R7" (id 0) (at 219.71 40.64 90))
-    (property "Value" "150k" (id 1) (at 219.71 43.18 90))
+    (property "Value" "15k" (id 1) (at 219.71 43.18 90))
     (property "Footprint" "Resistor_SMD:R_0805_2012Metric_Pad1.20x1.40mm_HandSolder" (id 2) (at 219.71 48.768 90)
       (effects (font (size 1.27 1.27)) hide)
