File: spinnybot-motherboad/connectors.kicad_sch (KiCad schematic)
At the start: 16 parts, among them J1 ENCODER 1, J12 LEDSTRIP3, J13 LEDSTRIP2, J14 LEDSTRIP3, J2 LEDSTRIP1, J3 LEDSTRIP1, J4 LEDSTRIP2, J5 ENCODER 2, J6 ENCODER 3, J7 SM10B-SRSS-TB

Commit message: Continued adding to board layout, added missing ESC connector footprint
Parts:
- J7: footprint CONN_SM10B-SRSS-TB_JST -> esc_4in1:SM10B-SRSS-TB
Changed lines of the file:
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@@
       (effects (font (size 1.524 1.524)))
     )
-    (property "Footprint" "CONN_SM10B-SRSS-TB_JST" (id 2) (at 149.86 79.756 0)
+    (property "Footprint" "esc_4in1:SM10B-SRSS-TB" (id 2) (at 149.86 79.756 0)
       (effects (font (size 1.524 1.524)) hide)
     )
